File: pcb/main.kicad_sch (KiCad schematic)
At the start: 13 parts, among them Q1 BC337, U1 LM358

Commit message: Placed all components.
Parts:
- added C10, C11, C12, C13, C17: 4n7, Capacitor_SMD:C_1206_3216Metric_Pad1.33x1.80mm_HandSolder, symbol Device:C
- added C14, C16, C2, C3, C4, C5: 1u, Capacitor_SMD:C_1206_3216Metric_Pad1.33x1.80mm_HandSolder, symbol Device:C
- added C15: 1n, Capacitor_SMD:C_1206_3216Metric_Pad1.33x1.80mm_HandSolder, symbol Device:C
- added D2, D3, D4, D5: 1N5817, Diode_THT:D_A-405_P10.16mm_Horizontal, symbol Device:D_Schottky
- added R10, R6, R7, R9: 15k, Resistor_SMD:R_1206_3216Metric_Pad1.30x1.75mm_HandSolder, symbol Device:R
- added R11, R8: 33k, Resistor_SMD:R_1206_3216Metric_Pad1.30x1.75mm_HandSolder, symbol Device:R
- added R12: 1k, Resistor_SMD:R_1206_3216Metric_Pad1.30x1.75mm_HandSolder, symbol Device:R
- added R13, R14, R15, R16, R17: 100k, deps:Trimmer 3362P, symbol Device:R_Trim
- added R18, R19: 100k, Resistor_SMD:R_1206_3216Metric_Pad1.30x1.75mm_HandSolder, symbol Device:R
- added RV4: 1k, deps:Potentiometer 3362P, symbol Device:R_Potentiometer
- added U2, U3, U4, U5, U6: LM358, Package_SO:SOIC-8_5.3x6.2mm_P1.27mm, symbol Amplifier_Operational:LM358
- U1: footprint (none) -> Package_SO:SOIC-8_5.3x6.2mm_P1.27mm
Connections:
- net +5V: now also RV4.1, U2.8 (V+), U3.8 (V+), U4.8 (V+), U5.8 (V+), U6.8 (V+)
- net GND: now also C15.2, C17.2, C2.2, C3.2, C4.2, C5.2, R10.2, R13.1, R18.2, R19.2, R7.2, U2.4 (V-), U3.4 (V-), U4.4 (V-), U4.5 (+), U5.4 (V-), U6.4 (V-), U6.6 (-)
- net at RV3.2, U1.5 (+): now also U2.2 (-), U2.6 (-)
- net at RV2.3, U1.7: now also R6.2
- new net: C4.1, C5.1, D5.1 (K), R19.1, U6.2 (-)
- new net: C2.1, C3.1, D4.1 (K), R18.1, U6.3 (+)
- new net: C17.1, R17.2, U5.5 (+)
- new net: C12.2, R11.1, R12.1, U2.7
- new net: C13.2, R11.2, U2.5 (+)
- new net: U4.6 (-), U4.7
- new net: C16.2, D5.2 (A), U5.6 (-), U5.7
- new net: R14.1, R16.1, U4.1, U4.2 (-)
- new net: C16.1, R16.2, R17.1
- new net: C14.2, D4.2 (A), U5.1, U5.2 (-)
- new net: C12.1, C13.1, R10.1, R9.1
- new net: D2.2 (A), D3.1 (K), R12.2, U3.2 (-), U3.6 (-), U4.3 (+)
- new net: D3.2 (A), U3.7
- new net: C15.1, R15.2, U5.3 (+)
- new net: D2.1 (K), U3.1
- new net: RV4.2, U3.3 (+)
- new net: R13.2, RV4.3, U3.5 (+)
- new net: C10.1, C11.1, R6.1, R7.1
- new net: C14.1, R14.2, R15.1
- new net: C11.2, R8.2, U2.3 (+)
- new net: C10.2, R8.1, R9.2, U2.1
- new net: U6.5 (+), U6.7
- new net signal: U6.1
Other:
- note added: "Amplifier for 2125Hz."
- note added: "Amplifier for 2295Hz."
- note added: "Clipping."
- note added: "Narrowband Filtering."
- note added: "Rectification & Differentiation."
- moved on the sheet: A1, C1, D1, Q1, R1, R2, R3, R4, R5, RV2, RV3, U1A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
